Commit message: refactor: move definition of URDF XACRO macros to different file

File: SoftTrunk/urdf/robot.urdf.xacro (robot description, xacro)
@@ -4,101 +4,10 @@
 -->
 <robot xmlns:xacro="http://www.ros.org/wiki/xacro" name="robot">
-  <material name="white">
-    <color rgba="1 1 1 1"/>
-  </material>
-  <xacro:macro name="ball_joint" params="id parent child">
-    <!--creates a ball joint.-->
-    <joint name="${parent}_${id}a_joint" type="revolute">
-      <parent link="${parent}"/>
-      <child link="${id}a"/>
-      <axis xyz="0 0 1"/>
-      <limit lower="-3.14" upper="3.14" effort="1000" velocity="1000"/>
-    </joint>
-    <link name="${id}a">
-      <visual>
-        <geometry>
-          <sphere radius="${length/20}"/>
-        </geometry>
-        <material name="white"/>
-      </visual>
-      <inertial>
-        <mass value="1"/>
-        <inertia ixx="1" ixy="1" ixz="1" iyy="1" iyz="1" izz="1"/>
-      </inertial>
-    </link>
-    <joint name="${id}a_${child}_joint" type="revolute">
-      <parent link="${id}a"/>
-      <child link="${child}"/>
-      <axis xyz="1 0 0"/>
-      <limit lower="-3.14" upper="3.14" effort="1000" velocity="1000"/>
-    </joint>
-  </xacro:macro>
-  <xacro:macro name="PCC" params="id parent child length">
-    <!--creates a PCC piece-->
-    <xacro:ball_joint id="${parent}_${id}a_balljoint" parent="${parent}" child="${id}a"/>
-    <link name="${id}a">
-      <inertial>
-        <mass value="1"/>
-        <inertia ixx="1" ixy="1" ixz="1" iyy="1" iyz="1" izz="1"/>
-      </inertial>
-    </link>
-    <joint name="${id}a_${id}b_joint" type="prismatic">
-      <parent link="${id}a"/>
-      <child link="${id}b"/>
-      <axis xyz="0 0 1"/>
-      <origin xyz="0 0 ${-length/2}"/>
-      <limit lower="0" upper="${length/2}" effort="1000" velocity="1000"/>
-    </joint>
-    <link name="${id}b">
-      <visual>
-        <geometry>
-          <sphere radius="${length/10}"/>
-        </geometry>
-        <material name="white"/>
-      </visual>
-      <inertial>
-        <mass value="1000"/>
-        <inertia ixx="1" ixy="1" ixz="1" iyy="1" iyz="1" izz="1"/>
-      </inertial>
-    </link>
-    <joint name="${id}b_${id}c_joint" type="prismatic">
-      <parent link="${id}b"/>
-      <child link="${id}c"/>
-      <axis xyz="0 0 1"/>
-      <origin xyz="0 0 ${-length/2}"/>
-      <limit lower="0" upper="${length/2}" effort="1000" velocity="1000"/>
-    </joint>
-    <link name="${id}c">
-      <inertial>
-        <mass value="1"/>
-        <inertia ixx="1" ixy="1" ixz="1" iyy="1" iyz="1" izz="1"/>
-      </inertial>
-    </link>
-    <xacro:ball_joint id="${id}c_${child}_balljoint" parent="${id}c" child="${child}"/>
-  </xacro:macro>
-  <link name="base_link">
-    <visual>
-      <geometry>
-        <box size="0.05 0.05 0.05" />
-        <material name="white"/>
-      </geometry>
-    </visual>
-    <inertial>
-      <mass value="1"/>
-      <inertia ixx="1" ixy="1" ixz="1" iyy="1" iyz="1" izz="1"/>
-    </inertial>
-  </link>
-  <xacro:PCC id="0" parent="base_link" child="end" length="0.5"/>
-  <link name="end">
-    <visual>
-      <geometry>
-        <box size="0.05 0.05 0.05" />
-        <material name="white"/>
-      </geometry>
-    </visual>
-    <inertial>
-      <mass value="1"/>
-      <inertia ixx="1" ixy="1" ixz="1" iyy="1" iyz="1" izz="1"/>
-    </inertial>
-  </link>
+  <xacro:include filename="macro_definitions.urdf.xacro" />
+  <xacro:empty_link name="base_link"/>
+  <xacro:PCC id="0" parent="base_link" child="0_mid" length="0.5"/>
+  <!--<xacro:PCC id="1" parent="0" child="end_link" length="0.5"/>-->
+  <xacro:empty_link name="0_mid"/>
+  <xacro:PCC id="1" parent="0_mid" child="end_link" length = "0.7" />
+  <xacro:empty_link name="end_link"/>
 </robot>
