Commit message: feat: PCC now reflects actual augmented model docs: how to create robot model

File: SoftTrunk/urdf/macro_definitions.urdf.xacro (robot description, xacro)
@@ -1,5 +1,5 @@
 <?xml version="1.0"?>
 <!--
-convert this to a URDF with $./create_urdf.sh
+this file defines the xacro macros that can be used to create PCC augmented models
 -->
 <robot xmlns:xacro="http://www.ros.org/wiki/xacro" name="robot">
@@ -7,26 +7,25 @@
     <color rgba="1 1 1 1"/>
   </material>
-  <xacro:macro name="ball_joint" params="id parent child">
-    <!--creates a ball joint.-->
-    <joint name="${parent}_${id}-a_joint" type="revolute">
+  <material name="red">
+    <color rgba="1 0 0 1"/>
+  </material>
+  <xacro:macro name="ball-joint" params="id parent child">
+    <!--creates a ball joint, called from the PCC macro..-->
+    <joint name="${id}-ball-joint_phi_joint" type="revolute">
       <parent link="${parent}"/>
-      <child link="${id}-a"/>
+      <child link="${id}-ball-joint_link"/>
       <axis xyz="0 0 1"/>
       <limit lower="-3.14" upper="3.14" effort="1000" velocity="1000"/>
     </joint>
-    <link name="${id}-a">
+    <link name="${id}-ball-joint_link">
       <visual>
         <geometry>
-          <sphere radius="${length/20}"/>
+          <box size="${length/10} ${length/10} ${length/10}"/>
         </geometry>
         <material name="white"/>
       </visual>
-      <inertial>
-        <mass value="1"/>
-        <inertia ixx="1" ixy="1" ixz="1" iyy="1" iyz="1" izz="1"/>
-      </inertial>
     </link>
-    <joint name="${id}-a_${child}_joint" type="revolute">
-      <parent link="${id}-a"/>
+    <joint name="${id}-ball-joint_theta_joint" type="revolute">
+      <parent link="${id}-ball-joint_link"/>
       <child link="${child}"/>
       <axis xyz="1 0 0"/>
@@ -34,14 +33,29 @@
     </joint>
   </xacro:macro>
-  <xacro:macro name="PCC" params="id parent child length">
+  <xacro:macro name="rod" params="length">
+    <!--creates a visual of a rod.-->
+    <visual>
+      <geometry>
+        <cylinder radius="${length/50}" length="${length/2}"/>
+      </geometry>
+      <material name="white"/>
+      <origin xyz="0 0 ${-length/4}"/>
+    </visual>
+  </xacro:macro>
+  <xacro:macro name="default_inertial">
+    <!--since the RBDL needs a inertial info for each link, just assign a really small value to links where we don't have to consider inertia.-->
+    <inertial>
+      <mass value="0.01"/>
+      <inertia ixx="0.01" ixy="0.01" ixz="0.01" iyy="0.01" iyz="0.01" izz="0.01"/>
+    </inertial>
+  </xacro:macro>
+  <xacro:macro name="PCC" params="id parent child length mass">
     <!--creates a PCC piece-->
-    <xacro:ball_joint id="${id}-root-balljoint" parent="${parent}" child="${id}-a"/>
+    <xacro:ball-joint id="${id}-base" parent="${parent}" child="${id}-a"/>
     <link name="${id}-a">
-      <inertial>
-        <mass value="1"/>
-        <inertia ixx="1" ixy="1" ixz="1" iyy="1" iyz="1" izz="1"/>
-      </inertial>
+      <xacro:default_inertial/>
+      <xacro:rod length="${length}"/>
     </link>
-    <joint name="${id}-a_${id}-b_joint" type="prismatic">
+    <joint name="${id}-a-b_joint" type="prismatic">
       <parent link="${id}-a"/>
       <child link="${id}-b"/>
@@ -51,42 +65,49 @@
     </joint>
     <link name="${id}-b">
+      <xacro:default_inertial/>
+    </link>
+    <joint name="${id}-b_c_joint" type="revolute">
+      <parent link="${id}-b"/>
+      <child link="${id}-c"/>
+      <limit lower="-3.14" upper="3.14" effort="1000" velocity="1000"/>
+      <axis xyz="0 0 1"/>
+    </joint>
+    <link name="${id}-c">
       <visual>
         <geometry>
-          <sphere radius="${length/10}"/>
+          <box size="${length/4} ${length/4} ${length/4}"/>
         </geometry>
-        <material name="white"/>
+        <material name="red"/>
       </visual>
       <inertial>
-        <mass value="1000"/>
+        <mass value="${mass}"/>
         <inertia ixx="1" ixy="1" ixz="1" iyy="1" iyz="1" izz="1"/>
       </inertial>
     </link>
-    <joint name="${id}-b_${id}-c_joint" type="prismatic">
-      <parent link="${id}-b"/>
-      <child link="${id}-c"/>
+    <joint name="${id}-c_d_joint" type="revolute">
+      <parent link="${id}-c"/>
+      <child link="${id}-d"/>
+      <limit lower="-3.14" upper="3.14" effort="1000" velocity="1000"/>
+      <axis xyz="0 0 1"/>
+    </joint>
+    <link name="${id}-d">
+      <xacro:default_inertial/>
+      <xacro:rod length="${length}"/>
+    </link>
+    <joint name="${id}-d-e_joint" type="prismatic">
+      <parent link="${id}-d"/>
+      <child link="${id}-e"/>
       <axis xyz="0 0 1"/>
       <origin xyz="0 0 ${-length/2}"/>
       <limit lower="0" upper="${length/2}" effort="1000" velocity="1000"/>
     </joint>
-    <link name="${id}-c">
-      <inertial>
-        <mass value="1"/>
-        <inertia ixx="1" ixy="1" ixz="1" iyy="1" iyz="1" izz="1"/>
-      </inertial>
+    <link name="${id}-e">
+      <xacro:default_inertial/>
     </link>
-    <xacro:ball_joint id="${id}-tip-balljoint" parent="${id}-c" child="${child}"/>
+    <xacro:ball-joint id="${id}-tip-balljoint" parent="${id}-e" child="${child}"/>
   </xacro:macro>
   <xacro:macro name="empty_link" params="name">
     <link name="${name}">
-      <visual>
-        <geometry>
-          <box size="0.05 0.05 0.05" />
-          <material name="white"/>
-        </geometry>
-      </visual>
-      <inertial>
-        <mass value="1"/>
-        <inertia ixx="1" ixy="1" ixz="1" iyy="1" iyz="1" izz="1"/>
-      </inertial>
+      <xacro:default_inertial/>
     </link>
   </xacro:macro>

File: SoftTrunk/urdf/robot.urdf.xacro (robot description, xacro)
@@ -6,8 +6,7 @@
   <xacro:include filename="macro_definitions.urdf.xacro" />
   <xacro:empty_link name="base_link"/>
-  <xacro:PCC id="0" parent="base_link" child="0_mid" length="0.5"/>
-  <!--<xacro:PCC id="1" parent="0" child="end_link" length="0.5"/>-->
+  <xacro:PCC id="0" parent="base_link" child="0_mid" length="0.5" mass="1000"/>
   <xacro:empty_link name="0_mid"/>
-  <xacro:PCC id="1" parent="0_mid" child="end_link" length = "0.7" />
+  <xacro:PCC id="1" parent="0_mid" child="end_link" length = "0.5" mass="1000" />
   <xacro:empty_link name="end_link"/>
 </robot>

Commit message: first attempt at isolating theta. alpha shows up as 0 so something's not right...

File: SoftTrunk/urdf/macro_definitions.urdf.xacro (robot description, xacro)
@@ -47,6 +47,6 @@
     <!--since the RBDL needs a inertial info for each link, just assign a really small value to links where we don't have to consider inertia.-->
     <inertial>
-      <mass value="0.01"/>
-      <inertia ixx="0.01" ixy="0.01" ixz="0.01" iyy="0.01" iyz="0.01" izz="0.01"/>
+      <mass value="0.00001"/>
+      <inertia ixx="0.00001" ixy="0.00001" ixz="0.00001" iyy="0.00001" iyz="0.00001" izz="0.00001"/>
     </inertial>
   </xacro:macro>

Commit message: fix: refactor: SoftArm doesn't need to have start() called. refactor: in Augmentedrigidarm, Jm and dJm are initialized at the very beginning rather than at beginning

File: SoftTrunk/urdf/macro_definitions.urdf.xacro (robot description, xacro)
@@ -10,4 +10,5 @@
     <color rgba="1 0 0 1"/>
   </material>
+  <xacro:property name="PI" value="3.1415" />
   <xacro:macro name="ball-joint" params="id parent child">
     <!--creates a ball joint, called from the PCC macro..-->
@@ -16,5 +17,5 @@
       <child link="${id}-ball-joint_link"/>
       <axis xyz="0 0 1"/>
-      <limit lower="-3.14" upper="3.14" effort="1000" velocity="1000"/>
+      <limit lower="${-PI*2}" upper="${PI*2}" effort="1000" velocity="1000"/>
     </joint>
     <link name="${id}-ball-joint_link">
@@ -30,6 +31,6 @@
       <parent link="${id}-ball-joint_link"/>
       <child link="${child}"/>
-      <axis xyz="1 0 0"/>
-      <limit lower="-3.14" upper="3.14" effort="1000" velocity="1000"/>
+      <axis xyz="0 1 0"/>
+      <limit lower="0" upper="${PI}" effort="1000" velocity="1000"/>
     </joint>
   </xacro:macro>
@@ -41,5 +42,5 @@
       </geometry>
       <material name="white"/>
-      <origin xyz="0 0 ${-length/4}"/>
+      <origin xyz="0 0 ${length/4}"/>
     </visual>
   </xacro:macro>
@@ -61,6 +62,6 @@
       <parent link="${id}-a"/>
       <child link="${id}-b"/>
-      <axis xyz="0 0 1"/>
-      <origin xyz="0 0 ${-length/2}"/>
+      <axis xyz="0 0 -1"/>
+      <origin xyz="0 0 ${length/2}"/>
       <limit lower="0" upper="${length/2}" effort="1000" velocity="1000"/>
     </joint>
@@ -71,5 +72,5 @@
       <parent link="${id}-b"/>
       <child link="${id}-c"/>
-      <limit lower="-3.14" upper="3.14" effort="1000" velocity="1000"/>
+      <limit lower="${-2*PI}" upper="0" effort="1000" velocity="1000"/>
       <axis xyz="0 0 1"/>
     </joint>
@@ -83,5 +84,5 @@
       <inertial>
         <mass value="${mass}"/>
-        <inertia ixx="1" ixy="1" ixz="1" iyy="1" iyz="1" izz="1"/>
+        <inertia ixx="0.0001" ixy="0.0001" ixz="0.0001" iyy="0.0001" iyz="0.0001" izz="0.0001"/>
       </inertial>
     </link>
@@ -89,5 +90,5 @@
       <parent link="${id}-c"/>
       <child link="${id}-d"/>
-      <limit lower="-3.14" upper="3.14" effort="1000" velocity="1000"/>
+      <limit lower="0" upper="${2*PI}" effort="1000" velocity="1000"/>
       <axis xyz="0 0 1"/>
     </joint>
@@ -99,6 +100,6 @@
       <parent link="${id}-d"/>
       <child link="${id}-e"/>
-      <axis xyz="0 0 1"/>
-      <origin xyz="0 0 ${-length/2}"/>
+      <axis xyz="0 0 -1"/>
+      <origin xyz="0 0 ${length/2}"/>
       <limit lower="0" upper="${length/2}" effort="1000" velocity="1000"/>
     </joint>

Commit message: fix: URDF actually describes augmented model links properly fix: in Augmentedrigidarm, xi, J and dJ correspond properly to URDF fix: in AugmentedRigidArm, results wonky when theta=0 -> adds small value when theta=0 refactor: don't have to call SoftArm.start() anymore. Simulation mode is also now possible.

File: SoftTrunk/urdf/macro_definitions.urdf.xacro (robot description, xacro)
@@ -33,4 +33,29 @@
       <axis xyz="0 1 0"/>
       <limit lower="0" upper="${PI}" effort="1000" velocity="1000"/>
+    </joint>
+  </xacro:macro>
+  <!-- todo: more elegant solution to accomodate two types of ball joints? -->
+    <xacro:macro name="ball-joint-below" params="id parent child">
+    <!--creates a ball joint, called from the PCC macro..-->
+    <joint name="${id}-ball-joint_theta_joint" type="revolute">
+      <parent link="${parent}"/>
+      <child link="${id}-ball-joint_link"/>
+      <axis xyz="0 1 0"/>
+      <limit lower="0" upper="${PI}" effort="1000" velocity="1000"/>
+    </joint>
+    <link name="${id}-ball-joint_link">
+      <xacro:default_inertial/>
+      <visual>
+        <geometry>
+          <box size="${length/10} ${length/10} ${length/10}"/>
+        </geometry>
+        <material name="white"/>
+      </visual>
+    </link>
+    <joint name="${id}-ball-joint_phi_joint" type="revolute">
+      <parent link="${id}-ball-joint_link"/>
+      <child link="${child}"/>
+      <axis xyz="0 0 1"/>
+      <limit lower="${-PI*2}" upper="${PI*2}" effort="1000" velocity="1000"/>
     </joint>
   </xacro:macro>
@@ -107,5 +132,5 @@
       <xacro:default_inertial/>
     </link>
-    <xacro:ball-joint id="${id}-tip-balljoint" parent="${id}-e" child="${child}"/>
+    <xacro:ball-joint-below id="${id}-tip-balljoint" parent="${id}-e" child="${child}"/>
   </xacro:macro>
   <xacro:macro name="empty_link" params="name">

Commit message: Bug fixes for augmented arm model! (#16)
* macro_definitions.urdf.xacro and AugmentedRigidArm.cpp was not properly formed, did not behave the way a PCC augmented model should
* ball joint at top and bottom are actually not the same. phi element should come near root for top ball joint, theta element should come near root for bottom ball joint.
* the arm was not pointed towards +z as it should have been (it was pointed other way around, since that was just more natural looking in rviz while making it)
* the augmented configuration's xi, Jm and dJm was not calculated properly in some places

File: SoftTrunk/urdf/macro_definitions.urdf.xacro (robot description, xacro)
@@ -10,4 +10,5 @@
     <color rgba="1 0 0 1"/>
   </material>
+  <xacro:property name="PI" value="3.1415" />
   <xacro:macro name="ball-joint" params="id parent child">
     <!--creates a ball joint, called from the PCC macro..-->
@@ -16,5 +17,5 @@
       <child link="${id}-ball-joint_link"/>
       <axis xyz="0 0 1"/>
-      <limit lower="-3.14" upper="3.14" effort="1000" velocity="1000"/>
+      <limit lower="${-PI*2}" upper="${PI*2}" effort="1000" velocity="1000"/>
     </joint>
     <link name="${id}-ball-joint_link">
@@ -30,6 +31,31 @@
       <parent link="${id}-ball-joint_link"/>
       <child link="${child}"/>
-      <axis xyz="1 0 0"/>
-      <limit lower="-3.14" upper="3.14" effort="1000" velocity="1000"/>
+      <axis xyz="0 1 0"/>
+      <limit lower="0" upper="${PI}" effort="1000" velocity="1000"/>
+    </joint>
+  </xacro:macro>
+  <!-- todo: more elegant solution to accomodate two types of ball joints? -->
+    <xacro:macro name="ball-joint-below" params="id parent child">
+    <!--creates a ball joint, called from the PCC macro..-->
+    <joint name="${id}-ball-joint_theta_joint" type="revolute">
+      <parent link="${parent}"/>
+      <child link="${id}-ball-joint_link"/>
+      <axis xyz="0 1 0"/>
+      <limit lower="0" upper="${PI}" effort="1000" velocity="1000"/>
+    </joint>
+    <link name="${id}-ball-joint_link">
+      <xacro:default_inertial/>
+      <visual>
+        <geometry>
+          <box size="${length/10} ${length/10} ${length/10}"/>
+        </geometry>
+        <material name="white"/>
+      </visual>
+    </link>
+    <joint name="${id}-ball-joint_phi_joint" type="revolute">
+      <parent link="${id}-ball-joint_link"/>
+      <child link="${child}"/>
+      <axis xyz="0 0 1"/>
+      <limit lower="${-PI*2}" upper="${PI*2}" effort="1000" velocity="1000"/>
     </joint>
   </xacro:macro>
@@ -41,5 +67,5 @@
       </geometry>
       <material name="white"/>
-      <origin xyz="0 0 ${-length/4}"/>
+      <origin xyz="0 0 ${length/4}"/>
     </visual>
   </xacro:macro>
@@ -61,6 +87,6 @@
       <parent link="${id}-a"/>
       <child link="${id}-b"/>
-      <axis xyz="0 0 1"/>
-      <origin xyz="0 0 ${-length/2}"/>
+      <axis xyz="0 0 -1"/>
+      <origin xyz="0 0 ${length/2}"/>
       <limit lower="0" upper="${length/2}" effort="1000" velocity="1000"/>
     </joint>
@@ -71,5 +97,5 @@
       <parent link="${id}-b"/>
       <child link="${id}-c"/>
-      <limit lower="-3.14" upper="3.14" effort="1000" velocity="1000"/>
+      <limit lower="${-2*PI}" upper="0" effort="1000" velocity="1000"/>
       <axis xyz="0 0 1"/>
     </joint>
@@ -83,5 +109,5 @@
       <inertial>
         <mass value="${mass}"/>
-        <inertia ixx="1" ixy="1" ixz="1" iyy="1" iyz="1" izz="1"/>
+        <inertia ixx="0.0001" ixy="0.0001" ixz="0.0001" iyy="0.0001" iyz="0.0001" izz="0.0001"/>
       </inertial>
     </link>
@@ -89,5 +115,5 @@
       <parent link="${id}-c"/>
       <child link="${id}-d"/>
-      <limit lower="-3.14" upper="3.14" effort="1000" velocity="1000"/>
+      <limit lower="0" upper="${2*PI}" effort="1000" velocity="1000"/>
       <axis xyz="0 0 1"/>
     </joint>
@@ -99,6 +125,6 @@
       <parent link="${id}-d"/>
       <child link="${id}-e"/>
-      <axis xyz="0 0 1"/>
-      <origin xyz="0 0 ${-length/2}"/>
+      <axis xyz="0 0 -1"/>
+      <origin xyz="0 0 ${length/2}"/>
       <limit lower="0" upper="${length/2}" effort="1000" velocity="1000"/>
     </joint>
@@ -106,5 +132,5 @@
       <xacro:default_inertial/>
     </link>
-    <xacro:ball-joint id="${id}-tip-balljoint" parent="${id}-e" child="${child}"/>
+    <xacro:ball-joint-below id="${id}-tip-balljoint" parent="${id}-e" child="${child}"/>
   </xacro:macro>
   <xacro:macro name="empty_link" params="name">

Commit message: feat: start converting to new parameterization (using deltaLa and deltaLb). phi-theta is not used anymore(except as temporary variables when calculating from Optitrack) feat: new augmented model (unverified on ROS, yet) feat: thanks to new parametrization, removed the phi PD controllers! feat: in order to calculate deltaLa and deltaLb, the radius of the soft trunk is defined in softtrunk_common_defs. feat: adaptable to 3 or 4 chambers (work in progress) feat: SoftArm.actuatePressure() takes pressure of all the chambers. feat: half-assed attempt at trying to convert to new augmented model, in AugmentedRigidArm. feat: just a single value used for k,d,alpha, for now.

File: SoftTrunk/urdf/macro_definitions.urdf.xacro (robot description, xacro)
@@ -13,8 +13,8 @@
   <xacro:macro name="ball-joint" params="id parent child">
     <!--creates a ball joint, called from the PCC macro..-->
-    <joint name="${id}-ball-joint_phi_joint" type="revolute">
+    <joint name="${id}-ball-joint_x_joint" type="revolute">
       <parent link="${parent}"/>
       <child link="${id}-ball-joint_link"/>
-      <axis xyz="0 0 1"/>
+      <axis xyz="1 0 0"/>
       <limit lower="${-PI*2}" upper="${PI*2}" effort="1000" velocity="1000"/>
     </joint>
@@ -28,34 +28,9 @@
       </visual>
     </link>
-    <joint name="${id}-ball-joint_theta_joint" type="revolute">
+    <joint name="${id}-ball-joint_y_joint" type="revolute">
       <parent link="${id}-ball-joint_link"/>
       <child link="${child}"/>
       <axis xyz="0 1 0"/>
       <limit lower="0" upper="${PI}" effort="1000" velocity="1000"/>
-    </joint>
-  </xacro:macro>
-  <!-- todo: more elegant solution to accomodate two types of ball joints? -->
-    <xacro:macro name="ball-joint-below" params="id parent child">
-    <!--creates a ball joint, called from the PCC macro..-->
-    <joint name="${id}-ball-joint_theta_joint" type="revolute">
-      <parent link="${parent}"/>
-      <child link="${id}-ball-joint_link"/>
-      <axis xyz="0 1 0"/>
-      <limit lower="0" upper="${PI}" effort="1000" velocity="1000"/>
-    </joint>
-    <link name="${id}-ball-joint_link">
-      <xacro:default_inertial/>
-      <visual>
-        <geometry>
-          <box size="${length/10} ${length/10} ${length/10}"/>
-        </geometry>
-        <material name="white"/>
-      </visual>
-    </link>
-    <joint name="${id}-ball-joint_phi_joint" type="revolute">
-      <parent link="${id}-ball-joint_link"/>
-      <child link="${child}"/>
-      <axis xyz="0 0 1"/>
-      <limit lower="${-PI*2}" upper="${PI*2}" effort="1000" velocity="1000"/>
     </joint>
   </xacro:macro>
@@ -92,13 +67,4 @@
     </joint>
     <link name="${id}-b">
-      <xacro:default_inertial/>
-    </link>
-    <joint name="${id}-b_c_joint" type="revolute">
-      <parent link="${id}-b"/>
-      <child link="${id}-c"/>
-      <limit lower="${-2*PI}" upper="0" effort="1000" velocity="1000"/>
-      <axis xyz="0 0 1"/>
-    </joint>
-    <link name="${id}-c">
       <visual>
         <geometry>
@@ -112,25 +78,15 @@
       </inertial>
     </link>
-    <joint name="${id}-c_d_joint" type="revolute">
-      <parent link="${id}-c"/>
-      <child link="${id}-d"/>
-      <limit lower="0" upper="${2*PI}" effort="1000" velocity="1000"/>
-      <axis xyz="0 0 1"/>
-    </joint>
-    <link name="${id}-d">
-      <xacro:default_inertial/>
-      <xacro:rod length="${length}"/>
-    </link>
-    <joint name="${id}-d-e_joint" type="prismatic">
-      <parent link="${id}-d"/>
-      <child link="${id}-e"/>
+    <joint name="${id}-b-c_joint" type="prismatic">
+      <parent link="${id}-b"/>
+      <child link="${id}-c"/>
       <axis xyz="0 0 -1"/>
       <origin xyz="0 0 ${length/2}"/>
       <limit lower="0" upper="${length/2}" effort="1000" velocity="1000"/>
     </joint>
-    <link name="${id}-e">
+    <link name="${id}-c">
       <xacro:default_inertial/>
     </link>
-    <xacro:ball-joint-below id="${id}-tip-balljoint" parent="${id}-e" child="${child}"/>
+    <xacro:ball-joint id="${id}-tip-balljoint" parent="${id}-c" child="${child}"/>
   </xacro:macro>
   <xacro:macro name="empty_link" params="name">

Commit message: fix: xacro macro_definition's joint limits and visuals

File: SoftTrunk/urdf/macro_definitions.urdf.xacro (robot description, xacro)
@@ -17,5 +17,5 @@
       <child link="${id}-ball-joint_link"/>
       <axis xyz="1 0 0"/>
-      <limit lower="${-PI*2}" upper="${PI*2}" effort="1000" velocity="1000"/>
+      <limit lower="${-PI/4}" upper="${PI/4}" effort="1000" velocity="1000"/>
     </joint>
     <link name="${id}-ball-joint_link">
@@ -32,8 +32,8 @@
       <child link="${child}"/>
       <axis xyz="0 1 0"/>
-      <limit lower="0" upper="${PI}" effort="1000" velocity="1000"/>
+      <limit lower="${-PI/4}" upper="${PI/4}" effort="1000" velocity="1000"/>
     </joint>
   </xacro:macro>
-  <xacro:macro name="rod" params="length">
+  <xacro:macro name="rod" params="length direction=1">
     <!--creates a visual of a rod.-->
     <visual>
@@ -42,5 +42,5 @@
       </geometry>
       <material name="white"/>
-      <origin xyz="0 0 ${length/4}"/>
+      <origin xyz="0 0 ${direction*length/4}"/>
     </visual>
   </xacro:macro>
@@ -87,4 +87,5 @@
     <link name="${id}-c">
       <xacro:default_inertial/>
+      <xacro:rod length="${length}" direction="-1"/>
     </link>
     <xacro:ball-joint id="${id}-tip-balljoint" parent="${id}-c" child="${child}"/>
