Commit message: feat: 11-DoF for each PCC segment feat: ROS publisher of joint states todo: don't do ROS stuff when it's not installed (how to do this??)

File: SoftTrunk/urdf/macro_definitions.urdf.xacro (robot description, xacro)
@@ -15,9 +15,18 @@
     <joint name="${id}-ball-joint_x_joint" type="revolute">
       <parent link="${parent}"/>
-      <child link="${id}-ball-joint_link"/>
+      <child link="${id}-ball-joint_link_0"/>
       <axis xyz="1 0 0"/>
       <limit lower="${-PI/4}" upper="${PI/4}" effort="1000" velocity="1000"/>
     </joint>
-    <link name="${id}-ball-joint_link">
+    <link name="${id}-ball-joint_link_0">
+      <xacro:default_inertial/>
+    </link>
+    <joint name="${id}-ball-joint_y_joint" type="revolute">
+      <parent link="${id}-ball-joint_link_0"/>
+      <child link="${id}-ball-joint_link_1"/>
+      <axis xyz="0 1 0"/>
+      <limit lower="${-PI/4}" upper="${PI/4}" effort="1000" velocity="1000"/>
+    </joint>
+    <link name="${id}-ball-joint_link_1">
       <xacro:default_inertial/>
       <visual>
@@ -28,8 +37,8 @@
       </visual>
     </link>
-    <joint name="${id}-ball-joint_y_joint" type="revolute">
-      <parent link="${id}-ball-joint_link"/>
+    <joint name="${id}-ball-joint_z_joint" type="revolute">
+      <parent link="${id}-ball-joint_link_1"/>
       <child link="${child}"/>
-      <axis xyz="0 1 0"/>
+      <axis xyz="0 0 1"/>
       <limit lower="${-PI/4}" upper="${PI/4}" effort="1000" velocity="1000"/>
     </joint>
@@ -78,16 +87,20 @@
       </inertial>
     </link>
-    <joint name="${id}-b-c_joint" type="prismatic">
-      <parent link="${id}-b"/>
-      <child link="${id}-c"/>
+    <xacro:ball-joint id="${id}-middle" parent="${id}-b" child="${id}-c"/>
+    <link name="${id}-c">
+      <xacro:default_inertial/>
+    </link>
+    <joint name="${id}-c-d_joint" type="prismatic">
+      <parent link="${id}-c"/>
+      <child link="${id}-d"/>
       <axis xyz="0 0 -1"/>
       <origin xyz="0 0 ${length/2}"/>
       <limit lower="0" upper="${length/2}" effort="1000" velocity="1000"/>
     </joint>
-    <link name="${id}-c">
+    <link name="${id}-d">
       <xacro:default_inertial/>
       <xacro:rod length="${length}" direction="-1"/>
     </link>
-    <xacro:ball-joint id="${id}-tip-balljoint" parent="${id}-c" child="${child}"/>
+    <xacro:ball-joint id="${id}-tip" parent="${id}-d" child="${child}"/>
   </xacro:macro>
   <xacro:macro name="empty_link" params="name">

Commit message: refactor ValveController to work mainly using actuator IDs instead of valve IDs, move more #define macros (bad) to const (good),

File: SoftTrunk/urdf/macro_definitions.urdf.xacro (robot description, xacro)
@@ -58,5 +58,5 @@
     <inertial>
       <mass value="0.00001"/>
-      <inertia ixx="0.00001" ixy="0.00001" ixz="0.00001" iyy="0.00001" iyz="0.00001" izz="0.00001"/>
+      <inertia ixx="0.00001" ixy="0.0000" ixz="0.0000" iyy="0.00001" iyz="0.0000" izz="0.00001"/>
     </inertial>
   </xacro:macro>
@@ -84,5 +84,5 @@
       <inertial>
         <mass value="${mass}"/>
-        <inertia ixx="0.0001" ixy="0.0001" ixz="0.0001" iyy="0.0001" iyz="0.0001" izz="0.0001"/>
+        <inertia ixx="0.0001" ixy="0.000" ixz="0.000" iyy="0.0001" iyz="0.000" izz="0.0001"/>
       </inertial>
     </link>
