Commit message: feat: update & visualize Drake model from PCC parameters q, feat: can set arm placement configuration

File: urdf/3segment_4chamber.urdf (robot description, URDF)
Before this commit: robot 3segment_4chamber, 23 links, 22 joints
Links:
- added link 2-a, mass 0.00001; visual cylinder length=0.055 radius=0.0022
- added link 2-b, mass 0.12; visual box size=0.0275 0.0275 0.0275
- added link 2-base-ball-joint_link_0, mass 0.00001
- added link 2-base-ball-joint_link_1, mass 0.00001; visual box size=0.011 0.011 0.011
- added link 2-c, mass 0.00001
- added link 2-d, mass 0.00001; visual cylinder length=0.055 radius=0.0022
- added link 2-middle-ball-joint_link_0, mass 0.00001
- added link 2-middle-ball-joint_link_1, mass 0.00001; visual box size=0.011 0.011 0.011
- added link 2-tip-ball-joint_link_0, mass 0.00001
- added link 2-tip-ball-joint_link_1, mass 0.00001; visual box size=0.011 0.011 0.011
- added link mid-2, mass 0.00001
Joints:
- added joint 2-a-b_joint: type prismatic, parent 2-a, child 2-b, origin xyz=0 0 0.055, axis 0 0 -1, limit lower=0 upper=0.055 effort=1000 velocity=1000
- added joint 2-base-ball-joint_x_joint: type revolute, parent mid-1, child 2-base-ball-joint_link_0, axis 1 0 0, limit lower=-0.785375 upper=0.785375 effort=1000 velocity=1000
- added joint 2-base-ball-joint_y_joint: type revolute, parent 2-base-ball-joint_link_0, child 2-base-ball-joint_link_1, axis 0 1 0, limit lower=-0.785375 upper=0.785375 effort=1000 velocity=1000
- added joint 2-base-ball-joint_z_joint: type revolute, parent 2-base-ball-joint_link_1, child 2-a, axis 0 0 1, limit lower=-0.785375 upper=0.785375 effort=1000 velocity=1000
- added joint 2-c-d_joint: type prismatic, parent 2-c, child 2-d, origin xyz=0 0 0.055, axis 0 0 -1, limit lower=0 upper=0.055 effort=1000 velocity=1000
- added joint 2-middle-ball-joint_x_joint: type revolute, parent 2-b, child 2-middle-ball-joint_link_0, axis 1 0 0, limit lower=-0.785375 upper=0.785375 effort=1000 velocity=1000
- added joint 2-middle-ball-joint_y_joint: type revolute, parent 2-middle-ball-joint_link_0, child 2-middle-ball-joint_link_1, axis 0 1 0, limit lower=-0.785375 upper=0.785375 effort=1000 velocity=1000
- added joint 2-middle-ball-joint_z_joint: type revolute, parent 2-middle-ball-joint_link_1, child 2-c, axis 0 0 1, limit lower=-0.785375 upper=0.785375 effort=1000 velocity=1000
- added joint 2-tip-ball-joint_x_joint: type revolute, parent 2-d, child 2-tip-ball-joint_link_0, axis 1 0 0, limit lower=-0.785375 upper=0.785375 effort=1000 velocity=1000
- added joint 2-tip-ball-joint_y_joint: type revolute, parent 2-tip-ball-joint_link_0, child 2-tip-ball-joint_link_1, axis 0 1 0, limit lower=-0.785375 upper=0.785375 effort=1000 velocity=1000
- added joint 2-tip-ball-joint_z_joint: type revolute, parent 2-tip-ball-joint_link_1, child mid-2, axis 0 0 1, limit lower=-0.785375 upper=0.785375 effort=1000 velocity=1000

File: urdf/3segment_4chamber.urdf.xacro (robot description, xacro)
@@ -8,3 +8,5 @@
 <xacro:PCC id='1' parent='mid-0' child='mid-1' length='0.11' mass='0.12'/>
 <xacro:empty_link name='mid-1'/>
+<xacro:PCC id='2' parent='mid-1' child='mid-2' length='0.11' mass='0.12'/>
+<xacro:empty_link name='mid-2'/>
 </robot>
